File: power.kicad_sch (KiCad schematic)
At the start: 10 parts, among them SW1 SW_SPST, U5 AMS1117-3.3

Commit message: updated infomration on schematic; started working on layout
Other:
- company: (none) -> Erick Zamora 
- title: (none) -> Miniature Sumo Robot 
Changed lines of the file:
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@@
 	(generator_version "9.0")
 	(paper "A5")
+	(title_block
+		(title "Miniature Sumo Robot ")
+		(date "2025-09-26")
+		(rev "A")
+		(company "Erick Zamora ")
+	)
 	(junction
 		(at 69.85 48.26)
