File: receiver.kicad_sch (KiCad schematic)
At the start: 0 parts

Commit message: added IR receiver circuit
Parts:
- added C3: C, symbol Device:C_Polarized
- added D3: LED, LED_SMD:LED_1210_3225Metric, symbol Device:LED
- added R3, R4: R, Resistor_SMD:R_1210_3225Metric, symbol Device:R
- added U6: TSOP38233, OptoDevice:Vishay_MINICAST-3Pin, symbol Interface_Optical:TSOP382xx
Connections:
- new net: D3.2 (A), R4.1
- new net: C3.1, R3.1, U6.3 (Vs)
- new net +3.3V: R3.2, R4.2
- new net GND: C3.2, U6.2 (GND)
- new net IR_RECEIVE: D3.1 (K), U6.1 (OUT)

Commit message: added more details to schematics
Parts:
- C3: value C -> 160pF
- R3: value R -> 10k
- R4: value R -> 1k
Changed lines of the file:
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@@
 			)
 		)
-		(property "Value" "C"
+		(property "Value" "160pF"
 			(at 84.328 52.324 0)
 			(effects
@@
 			)
 		)
-		(property "Value" "R"
+		(property "Value" "10k"
 			(at 99.06 54.61 90)
 			(effects
@@
 		(dnp no)
 		(property "Reference" "R4"
-			(at 106.68 67.564 90)
-			(effects
-				(font
-					(size 1.27 1.27)
-				)
-			)
-		)
-		(property "Value" "R"
 			(at 106.68 65.786 90)
 			(effects
 				(font
+					(size 1.27 1.27)
+				)
+			)
+		)
+		(property "Value" "1k"
+			(at 107.188 67.564 90)
+			(effects
+				(font

Commit message: updated logic for MCU
Changed lines of the file:
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@@
 	(generator_version "9.0")
 	(paper "A5")
-	(text_box "Need to update R3 and C3 values "
-		(exclude_from_sim no)
-		(at 48.26 30.48 0)
-		(size 13.97 11.43)
-		(margins 0.9525 0.9525 0.9525 0.9525)
-		(stroke
-			(width 0)
-			(type solid)
-		)
-		(fill
-			(type none)
-		)
-		(effects
-			(font
-				(size 1.27 1.27)
-			)
-			(justify left top)
-		)
-	)
 	(junction
 		(at 87.63 58.42)

Commit message: added all footprints and step files to components
Parts:
- C3: footprint (none) -> Capacitor_SMD:C_1210_3225Metric
Changed lines of the file:
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@@
 			)
 		)
-		(property "Footprint" ""
+		(property "Footprint" "Capacitor_SMD:C_1210_3225Metric"
 			(at 86.6648 48.26 0)
 			(effects

Commit message: updated infomration on schematic; started working on layout
Other:
- company: (none) -> Erick Zamora 
- title: (none) -> Miniature Sumo Robot 
Changed lines of the file:
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@@
 	(generator_version "9.0")
 	(paper "A5")
+	(title_block
+		(title "Miniature Sumo Robot ")
+		(date "2025-09-26")
+		(rev "A")
+		(company "Erick Zamora ")
+	)
 	(junction
 		(at 87.63 58.42)
