File: micro.kicad_sch (KiCad schematic)
At the start: 21 parts, among them J15 Conn_01x02, J16 Conn_01x03, J17 Conn_01x08, J18 Conn_01x02, J19 Conn_01x02, SW3 SW_Omron_B3FS

Commit message: continued layout
Parts:
- H1, H2, H3, H4: footprint MountingHole:MountingHole_4.5mm_Pad -> MountingHole:MountingHole_2.5mm_Pad
Changed lines of the file:
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@@
 			)
 		)
-		(property "Footprint" "MountingHole:MountingHole_4.5mm_Pad"
+		(property "Footprint" "MountingHole:MountingHole_2.5mm_Pad"
 			(at 17.78 71.12 0)
 			(effects
@@
 			)
 		)
-		(property "Footprint" "MountingHole:MountingHole_4.5mm_Pad"
+		(property "Footprint" "MountingHole:MountingHole_2.5mm_Pad"
 			(at 17.78 83.82 0)
 			(effects
@@
 			)
 		)
-		(property "Footprint" "MountingHole:MountingHole_4.5mm_Pad"
+		(property "Footprint" "MountingHole:MountingHole_2.5mm_Pad"
 			(at 17.78 90.17 0)
 			(effects
@@
 			)
 		)
-		(property "Footprint" "MountingHole:MountingHole_4.5mm_Pad"
+		(property "Footprint" "MountingHole:MountingHole_2.5mm_Pad"
 			(at 17.78 77.47 0)
 			(effects

Commit message: updated infomration on schematic; started working on layout
Other:
- company: (none) -> Erick Zamora 
- title: (none) -> Miniature Sumo Robot 
Changed lines of the file:
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@@
 	(generator_version "9.0")
 	(paper "A5")
+	(title_block
+		(title "Miniature Sumo Robot ")
+		(date "2025-09-26")
+		(rev "A")
+		(company "Erick Zamora ")
+	)
 	(junction
 		(at 163.83 22.86)

Commit message: rethinking the layout
Parts:
- removed J17: Conn_01x08, Connector_PinHeader_1.00mm:PinHeader_1x08_P1.00mm_Vertical, symbol Connector_Generic:Conn_01x08
Connections:
- net UNUSED_1: no longer names the net of U1.16 (P2.3/TA1.0)
- net UNUSED_2: no longer names the net of U1.15 (P3.4/TA0.0)
- net UNUSED_3: no longer names the net of U1.8 (P3.1/TA1.0)
- net UNUSED_4: no longer names the net of U1.9 (P3.0/TA0.2)
- net UNUSED_5: no longer names the net of U1.11 (P2.1/TA1.1)
- net UNUSED_6: no longer names the net of U1.12 (P2.2/TA1.1)
- net UNUSED_7: no longer names the net of U1.13 (P3.2/TA1.1)
- net UNUSED_8: no longer names the net of U1.14 (P3.3/TA1.2)
- no-connect marks 0 -> 8
Other:
- moved on the sheet: R11, R12

Commit message: updating pcb layout
Parts:
- removed J15: Conn_01x02, Connector_PinHeader_1.00mm:PinHeader_1x02_P1.00mm_Vertical, symbol Connector_Generic:Conn_01x02
Changed lines of the file:
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@@
 	)
 	(junction
-		(at 163.83 22.86)
-		(diameter 0)
-		(color 0 0 0 0)
-	)
-	(junction
 		(at 175.26 92.71)
 		(diameter 0)
@@
 	(wire
 		(pts
-			(xy 171.45 31.75) (xy 171.45 35.56)
-		)
-		(stroke
-			(width 0)
-			(type default)
-		)
-	)
-	(wire
-		(pts
 			(xy 137.16 86.36) (xy 143.51 86.36)
 		)
@@
 	(wire
 		(pts
-			(xy 163.83 22.86) (xy 158.75 22.86)
-		)
-		(stroke
-			(width 0)
-			(type default)
-		)
-	)
-	(wire
-		(pts
 			(xy 163.83 63.5) (xy 163.83 68.58)
 		)
@@
 	(wire
 		(pts
-			(xy 168.91 22.86) (xy 163.83 22.86)
-		)
-		(stroke
-			(width 0)
-			(type default)
-		)
-	)
-	(wire
-		(pts
 			(xy 58.42 66.04) (xy 58.42 68.58)
 		)
@@
 	(wire
 		(pts
-			(xy 163.83 21.59) (xy 163.83 22.86)
-		)
-		(stroke
-			(width 0)
-			(type default)
-		)
-	)
-	(wire
-		(pts
-			(xy 158.75 22.86) (xy 158.75 24.13)
+			(xy 158.75 21.59) (xy 158.75 24.13)
 		)
 		(stroke
@@
 	(wire
 		(pts
-			(xy 168.91 35.56) (xy 168.91 22.86)
-		)
-		(stroke
-			(width 0)
-			(type default)
-		)
-	)
-	(wire
-		(pts
 			(xy 137.16 66.04) (xy 143.51 66.04)
 		)
@@
 	(global_label "TEST_LED"
 		(shape output)
-		(at 163.83 21.59 90)
+		(at 158.75 21.59 90)
 		(fields_autoplaced yes)
 		(effects
@@
 		)
 		(property "Intersheetrefs" "${INTERSHEET_REFS}"
-			(at 163.83 13.4046 90)
+			(at 158.75 13.4046 90)
 			(effects
 				(font
@@
 	)
 	(symbol
-		(lib_id "power:GND")
-		(at 171.45 31.75 180)
-		(unit 1)
-		(exclude_from_sim no)
-		(in_bom yes)
-		(on_board yes)
-		(dnp no)
-		(fields_autoplaced yes)
-		(property "Reference" "#PWR055"
-			(at 171.45 25.4 0)
-			(effects
-				(font
-					(size 1.27 1.27)
-				)
-				(hide yes)
-			)
-		)
-		(property "Value" "GND"
-			(at 171.45 26.67 0)
-			(effects
-				(font
-					(size 1.27 1.27)
-				)
-			)
-		)
-		(property "Footprint" ""
-			(at 171.45 31.75 0)
-			(effects
-				(font
-					(size 1.27 1.27)
-				)
-				(hide yes)
-			)
-		)
-		(property "Datasheet" ""
-			(at 171.45 31.75 0)
-			(effects
-				(font
-					(size 1.27 1.27)
-				)
-				(hide yes)
-			)
-		)
-		(property "Description" "Power symbol creates a global label with name \"GND\" , ground"
-			(at 171.45 31.75 0)
-			(effects
-				(font
-					(size 1.27 1.27)
-				)
-				(hide yes)
-			)
-		)
-		(pin "1"
-		)
-		(instances
-			(project "Sumo_Robot"
-				(path "/f283bc71-7763-4093-b75c-cbe2f5868c12/9428f158-f7fc-4e4a-b97b-e16df299d57c"
-					(reference "#PWR055")
-					(unit 1)
-				)
-			)
-		)
-	)
-	(symbol
 		(lib_id "Mechanical:MountingHole")
 		(at 17.78 83.82 0)
@@
 					(unit 1)
 				)
-			)
-		)
-	)
-	(symbol
-		(lib_id "Connector_Generic:Conn_01x02")
-		(at 171.45 40.64 270)
-		(unit 1)
-		(exclude_from_sim no)
-		(in_bom yes)
-		(on_board yes)
-		(dnp no)
-		(property "Reference" "J15"
-			(at 168.656 43.434 90)
-			(effects
-				(font
-					(size 1.27 1.27)
-				)
-				(justify left)
-			)
-		)
-		(property "Value" "Conn_01x02"
-			(at 173.99 41.9099 90)
-			(effects
-				(font
-					(size 1.27 1.27)
-				)
-				(justify left)
-				(hide yes)
-			)
-		)
-		(property "Footprint" "Connector_PinHeader_1.00mm:PinHeader_1x02_P1.00mm_Vertical"
-			(at 171.45 40.64 0)
-			(effects
-				(font
-					(size 1.27 1.27)
-				)
-				(hide yes)
-			)
-		)
-		(property "Datasheet" "~"
-			(at 171.45 40.64 0)
-			(effects
-				(font
-					(size 1.27 1.27)
-				)
-				(hide yes)
-			)
-		)
-		(property "Description" "Generic connector, single row, 01x02, script generated (kicad-library-utils/schlib/autogen/connector/)"
-			(at 171.45 40.64 0)
-			(effects
-				(font
-					(size 1.27 1.27)
-				)
-				(hide yes)
-			)
-		)
-		(pin "1"
-		)
-		(pin "2"
-		)
-		(instances
-			(project ""
-				(path "/f283bc71-7763-4093-b75c-cbe2f5868c12/9428f158-f7fc-4e4a-b97b-e16df299d57c"
-					(reference "J15")
-					(unit 1)
-				)
